File: PCB/STM32L052K8T6-MCU.sch (KiCad schematic (older format))
At the start: 0 parts

Commit message: Spec Changes and Schematic
Tiny bit of progress on the schematic and change to the feature set. The
sub 1GHZ radio is going to be integrated into the same board as the
beagle sip, I'm doing away with the USB hub for now. Doing away with the
wireless chip from Ti going to use a ESP32 as a realtime controller and
for standard wireless since the focus is remote wireless not indoor
wireless. Need to fit all the important stuff first before adding extra
features like a USB hub.
Other:
- note removed: "Beaglebone Pink Wireless"
Changed lines of the file:
@@
 $Descr A4 11693 8268
 encoding utf-8
-Sheet 1 5
+Sheet 1 6
 Title ""
-Date "2016-10-16"
-Rev "0.1a"
-Comp "GhostPCB"
-Comment1 "Engineer Drawn By Adam Vadala-Roth"
-Comment2 "Designed By Adam Vadala-Roth"
+Date ""
+Rev ""
+Comp ""
+Comment1 ""
+Comment2 ""
 Comment3 ""
 Comment4 ""
 $EndDescr
-Text Notes 3100 1100 0    315  ~ 63
-Beaglebone Pink Wireless
-$Sheet
-S 7000 3375 2800 1475
-U 58040242
-F0 "Power" 60
-F1 "Power.sch" 60
-$EndSheet
-$Sheet
-S 1500 1475 1800 1400
-U 5804022F
-F0 "Beaglebone System In Package" 60
-F1 "SiP_OSD3358.sch" 60
-$EndSheet
-$Sheet
-S 7000 1450 2800 1425
-U 580402EF
-F0 "USB Connectivity" 60
-F1 "USB_Hub.sch" 60
-$EndSheet
-$Sheet
-S 1475 3575 2250 2000
-U 5882F261
-F0 "RF Transceiver - ADF7023" 60
-F1 "RF-Transceiver-ADF7023.sch" 60
-$EndSheet
 $EndSCHEMATC
